File: precharge.kicad_sch (KiCad schematic)
At the start: 12 parts, among them Q2 2N7000, Q3 2N7002, Q4 BC327

Commit message: echtes pcb
Parts:
- removed Q4: BC327, Package_TO_SOT_THT:TO-92_Inline, symbol Transistor_BJT:BC327
- added Q1: BC807, Package_TO_SOT_SMD:SOT-23, symbol Transistor_BJT:BC807
- C1: footprint Capacitor_SMD:C_1206_3216Metric_Pad1.33x1.80mm_HandSolder -> Capacitor_SMD:C_0805_2012Metric_Pad1.18x1.45mm_HandSolder
- D1: footprint (none) -> Diode_SMD:D_MiniMELF_Handsoldering
- D4: footprint Diode_THT:D_DO-35_SOD27_P7.62mm_Horizontal -> Diode_SMD:D_SOD-123; symbol Diode:1N4148 -> Diode:1N4148W
- Q2: footprint Package_TO_SOT_THT:TO-92_Inline -> Package_TO_SOT_SMD:SOT-23; symbol Transistor_FET:2N7000 -> Transistor_FET:2N7002
- R1, R4: footprint Resistor_SMD:R_2512_6332Metric_Pad1.40x3.35mm_HandSolder -> Resistor_THT:R_Axial_DIN0207_L6.3mm_D2.5mm_P10.16mm_Horizontal
- R2, R3: footprint Resistor_SMD:R_1206_3216Metric_Pad1.30x1.75mm_HandSolder -> Resistor_SMD:R_0805_2012Metric_Pad1.20x1.40mm_HandSolder
- R5: footprint Resistor_THT:R_Axial_DIN0204_L3.6mm_D1.6mm_P7.62mm_Horizontal -> Resistor_SMD:R_0805_2012Metric_Pad1.20x1.40mm_HandSolder
Connections:
- net Bat-: now also Q2.2 (S); no longer Q2.1 (S)
- net Gate_main: now also Q1.3 (C)
- net Main_SW: now also Q2.1 (G), Q1.2 (E); no longer Q2.2 (G)
Changed lines of the file:
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@@
   (junction (at 72.39 114.3) (diameter 0) (color 0 0 0 0)
   )
-  (junction (at 96.52 104.14) (diameter 0) (color 0 0 0 0)
-  )
   (junction (at 72.39 104.14) (diameter 0) (color 0 0 0 0)
   )
@@
     (stroke (width 0) (type default))
   )
-  (wire (pts (xy 96.52 101.6) (xy 96.52 104.14))
+  (wire (pts (xy 96.52 101.6) (xy 96.52 106.68))
     (stroke (width 0) (type default))
   )
@@
   )
   (wire (pts (xy 88.9 99.06) (xy 88.9 91.44))
-    (stroke (width 0) (type default))
-  )
-  (wire (pts (xy 96.52 104.14) (xy 96.52 106.68))
     (stroke (width 0) (type default))
   )
@@
       (effects (font (size 1.27 1.27)) (justify right))
     )
-    (property "Footprint" "Resistor_SMD:R_1206_3216Metric_Pad1.30x1.75mm_HandSolder" (at 98.298 97.79 90)
+    (property "Footprint" "Resistor_SMD:R_0805_2012Metric_Pad1.20x1.40mm_HandSolder" (at 98.298 97.79 90)
       (effects (font (size 1.27 1.27)) hide)
     )
@@
     )
   )
-  (symbol (lib_id "Diode:1N4148") (at 96.52 119.38 90) (unit 1)
+  (symbol (lib_id "Diode:1N4148W") (at 96.52 119.38 90) (unit 1)
     (in_bom yes) (on_board yes) (dnp no) (fields_autoplaced)
     (property "Reference" "D4" (at 99.06 118.11 90)
@@
       (effects (font (size 1.27 1.27)) (justify right))
     )
-    (property "Footprint" "Diode_THT:D_DO-35_SOD27_P7.62mm_Horizontal" (at 96.52 119.38 0)
-      (effects (font (size 1.27 1.27)) hide)
-    )
-    (property "Datasheet" "https://assets.nexperia.com/documents/data-sheet/1N4148_1N4448.pdf" (at 96.52 119.38 0)
+    (property "Footprint" "Diode_SMD:D_SOD-123" (at 100.965 119.38 0)
+      (effects (font (size 1.27 1.27)) hide)
+    )
+    (property "Datasheet" "https://www.vishay.com/docs/85748/1n4148w.pdf" (at 96.52 119.38 0)
       (effects (font (size 1.27 1.27)) hide)
     )
@@
       (effects (font (size 1.27 1.27)))
     )
-    (property "Footprint" "Resistor_SMD:R_2512_6332Metric_Pad1.40x3.35mm_HandSolder" (at 86.36 135.128 90)
+    (property "Footprint" "Resistor_THT:R_Axial_DIN0207_L6.3mm_D2.5mm_P10.16mm_Horizontal" (at 86.36 135.128 90)
       (effects (font (size 1.27 1.27)) hide)
     )
@@
       (effects (font (size 1.27 1.27)) (justify left))
     )
-    (property "Footprint" "" (at 96.52 128.27 0)
+    (property "Footprint" "Diode_SMD:D_MiniMELF_Handsoldering" (at 96.52 128.27 0)
       (effects (font (size 1.27 1.27)) hide)
     )
@@
     )
   )
-  (symbol (lib_id "Transistor_BJT:BC327") (at 91.44 104.14 180) (unit 1)
+  (symbol (lib_id "Transistor_BJT:BC807") (at 86.36 104.14 0) (mirror x) (unit 1)
     (in_bom yes) (on_board yes) (dnp no)
-    (property "Reference" "Q4" (at 86.36 105.41 0)
+    (property "Reference" "Q1" (at 91.44 105.41 0)
       (effects (font (size 1.27 1.27)) (justify left))
     )
-    (property "Value" "BC327" (at 86.36 102.87 0)
+    (property "Value" "BC807" (at 91.44 102.87 0)
       (effects (font (size 1.27 1.27)) (justify left))
     )
-    (property "Footprint" "Package_TO_SOT_THT:TO-92_Inline" (at 86.36 102.235 0)
+    (property "Footprint" "Package_TO_SOT_SMD:SOT-23" (at 91.44 102.235 0)
       (effects (font (size 1.27 1.27) italic) (justify left) hide)
     )
-    (property "Datasheet" "http://www.onsemi.com/pub_link/Collateral/BC327-D.PDF" (at 91.44 104.14 0)
+    (property "Datasheet" "https://www.onsemi.com/pub/Collateral/BC808-D.pdf" (at 86.36 104.14 0)
       (effects (font (size 1.27 1.27)) (justify left) hide)
     )
@@
       (project "precharge"
         (path "/f9c0b950-8ca0-4171-885e-62cd91d7ac2f"
-          (reference "Q4") (unit 1)
+          (reference "Q1") (unit 1)
         )
       )
@@
       (effects (font (size 1.27 1.27)) (justify right))
     )
-    (property "Footprint" "Resistor_THT:R_Axial_DIN0204_L3.6mm_D1.6mm_P7.62mm_Horizontal" (at 98.298 110.49 90)
+    (property "Footprint" "Resistor_SMD:R_0805_2012Metric_Pad1.20x1.40mm_HandSolder" (at 98.298 110.49 90)
       (effects (font (size 1.27 1.27)) hide)
     )
@@
       (effects (font (size 1.27 1.27)))
     )
-    (property "Footprint" "Resistor_SMD:R_2512_6332Metric_Pad1.40x3.35mm_HandSolder" (at 86.36 151.638 90)
+    (property "Footprint" "Resistor_THT:R_Axial_DIN0207_L6.3mm_D2.5mm_P10.16mm_Horizontal" (at 86.36 151.638 90)
       (effects (font (size 1.27 1.27)) hide)
     )
@@
       (effects (font (size 1.27 1.27)))
     )
-    (property "Footprint" "Resistor_SMD:R_1206_3216Metric_Pad1.30x1.75mm_HandSolder" (at 63.5 126.238 90)
+    (property "Footprint" "Resistor_SMD:R_0805_2012Metric_Pad1.20x1.40mm_HandSolder" (at 63.5 126.238 90)
       (effects (font (size 1.27 1.27)) hide)
     )
@@
     )
   )
-  (symbol (lib_id "Transistor_FET:2N7000") (at 72.39 130.81 270) (unit 1)
+  (symbol (lib_id "Transistor_FET:2N7002") (at 72.39 130.81 270) (unit 1)
     (in_bom yes) (on_board yes) (dnp no) (fields_autoplaced)
     (property "Reference" "Q2" (at 72.39 137.16 90)
@@
       (effects (font (size 1.27 1.27)))
     )
-    (property "Footprint" "Package_TO_SOT_THT:TO-92_Inline" (at 70.485 135.89 0)
+    (property "Footprint" "Package_TO_SOT_SMD:SOT-23" (at 70.485 135.89 0)
       (effects (font (size 1.27 1.27) italic) (justify left) hide)
     )
-    (property "Datasheet" "https://www.vishay.com/docs/70226/70226.pdf" (at 72.39 130.81 0)
+    (property "Datasheet" "https://www.onsemi.com/pub/Collateral/NDS7002A-D.PDF" (at 72.39 130.81 0)
       (effects (font (size 1.27 1.27)) (justify left) hide)
     )
@@
       (effects (font (size 1.27 1.27)))
     )
-    (property "Footprint" "Capacitor_SMD:C_1206_3216Metric_Pad1.33x1.80mm_HandSolder" (at 67.31 103.1748 0)
-      (effects (font (size 1.27 1.27)) hide)
-    )
+    (property "Footprint" "Capacitor_SMD:C_0805_2012Metric_Pad1.18x1.45mm_HandSolder" (at 67.31 103.1748 0)
+      (effects (font (size 1.27 1.27)) hide)
+    )
